Commit message: fine-tuning urdf collision geometry

File: tm_description/urdf/tm12s.urdf.xacro (robot description, xacro)
@@ -42,7 +42,7 @@
         <collision>
             <geometry>
-                <cylinder length="0.16" radius="0.095" />
-            </geometry>
-            <origin xyz="0 0 0.08" rpy="0 0 0" />
+                <cylinder length="0.07" radius="0.105" />
+            </geometry>
+            <origin xyz="0 0 0.035" rpy="0 0 0" />
         </collision>
     </link>
@@ -115,5 +115,5 @@
         <collision>
             <geometry>
-                <cylinder length="0.175" radius="0.076" />
+                <cylinder length="0.18" radius="0.075" />
             </geometry>
             <origin xyz="0.6361 0 0" rpy="0 0 0" />
@@ -149,5 +149,5 @@
         <collision>
         <geometry>
-            <cylinder length="0.1" radius="0.075" />
+            <cylinder length="0.09" radius="0.075" />
         </geometry>
         <origin xyz="0 0 0" rpy="0 0 0" />
@@ -161,5 +161,5 @@
         <collision>
         <geometry>
-            <cylinder length="0.136" radius="0.047" />
+            <cylinder length="0.131" radius="0.047" />
         </geometry>
         <origin xyz="0.5324 0 0" rpy="0 0 0" />
@@ -192,5 +192,5 @@
             <cylinder length="0.116" radius="0.047" />
         </geometry>
-        <origin xyz="0 0.007 0" rpy="${0.5*pi} 0 0" />
+        <origin xyz="0 0.01 0" rpy="${0.5*pi} 0 0" />
         </collision>
     </link>
@@ -224,7 +224,7 @@
         <collision>
         <geometry>
-            <cylinder length="0.14" radius="0.047" />
-        </geometry>
-        <origin xyz="0 0 0.0" rpy="0 0 0" />
+            <cylinder length="${wrist_3_length}" radius="0.047" />
+        </geometry>
+        <origin xyz="0 0 0.004" rpy="0 0 0" />
         </collision>
         <collision>
@@ -232,5 +232,5 @@
             <cylinder length="0.200" radius="0.047" />
         </geometry>
-        <origin xyz="0 -0.09 0" rpy="${0.5*pi} 0 0" />
+        <origin xyz="0 -0.095 0" rpy="${0.5*pi} 0 0" />
         </collision>
     </link>
