Commit message: added mesh/urdf version without camera

File: tm_description/urdf/tm1100.urdf.xacro (robot description, xacro)
@@ -230,5 +230,10 @@
       <visual>
         <geometry>
-	  <mesh filename="package://tm_description/meshes/tm1100/visual/Wrist3.STL" />
+          <xacro:if value="${has_camera}">
+          <mesh filename="package://tm_description/meshes/tm1100/visual/Wrist3.STL" />
+          </xacro:if>
+          <xacro:unless value="${has_camera}">
+          <mesh filename="package://tm_description/meshes/tm1100/visual/Wrist3_no_camera.STL" />
+          </xacro:unless>
         </geometry>
 	<origin xyz="0 0 0.015" rpy="0 0 0"/>
@@ -239,5 +244,10 @@
       <collision>
         <geometry>
-	  <mesh filename="package://tm_description/meshes/tm1100/collision/wrist_3.STL" />
+          <xacro:if value="${has_camera}">
+	      <mesh filename="package://tm_description/meshes/tm1100/collision/wrist_3.STL" />
+          </xacro:if>
+          <xacro:unless value="${has_camera}">
+	      <mesh filename="package://tm_description/meshes/tm1100/collision/wrist_3_no_camera.STL" />
+          </xacro:unless>
         </geometry>
       </collision>

File: tm_description/urdf/tm1100_robot.urdf.xacro (robot description, xacro)
@@ -8,5 +8,5 @@
   <!-- tm1100 -->
   <xacro:include filename="$(find tm_description)/urdf/tm1100.urdf.xacro" />
-  <xacro:tm1100_robot prefix="${prefix}" joint_limited="false" />
+  <xacro:tm1100_robot prefix="${prefix}" joint_limited="false" has_camera="true" />
   <link name="world" />
   <joint name="world_joint" type="fixed">

File: tm_description/urdf/tm1100_robot_joint_limited.urdf.xacro (robot description, xacro)
@@ -8,5 +8,5 @@
   <!-- tm1100 -->
   <xacro:include filename="$(find tm_description)/urdf/tm1100.urdf.xacro" />
-  <xacro:tm1100_robot prefix="${prefix}" joint_limited="true" />
+  <xacro:tm1100_robot prefix="${prefix}" joint_limited="true" has_camera="true" />
   <link name="world" />
   <joint name="world_joint" type="fixed">

File: tm_description/urdf/tm1300.urdf.xacro (robot description, xacro)
@@ -50,5 +50,5 @@
     </inertial>
   </xacro:macro>
-  <xacro:macro name="tm1300_robot" params="prefix joint_limited">
+  <xacro:macro name="tm1300_robot" params="prefix joint_limited has_camera">
     <!-- transmission prefix -->
     <xacro:tm_arm_transmission prefix="${prefix}" />
@@ -229,5 +229,10 @@
       <visual>
         <geometry>
-	  <mesh filename="package://tm_description/meshes/tm1300/visual/Wrist3.STL" />
+          <xacro:if value="${has_camera}">
+          <mesh filename="package://tm_description/meshes/tm1300/visual/Wrist3.STL" />
+          </xacro:if>
+          <xacro:unless value="${has_camera}">
+          <mesh filename="package://tm_description/meshes/tm1300/visual/Wrist3_no_camera.STL" />
+          </xacro:unless>
         </geometry>
 	<origin xyz="0 0 0.015" rpy="0 0 0"/>
@@ -238,5 +243,10 @@
       <collision>
         <geometry>
-	  <mesh filename="package://tm_description/meshes/tm1300/collision/wrist_3.STL" />
+          <xacro:if value="${has_camera}">
+	      <mesh filename="package://tm_description/meshes/tm1300/collision/wrist_3.STL" />
+          </xacro:if>
+          <xacro:unless value="${has_camera}">
+	      <mesh filename="package://tm_description/meshes/tm1300/collision/wrist_3_no_camera.STL" />
+          </xacro:unless>
         </geometry>
       </collision>

File: tm_description/urdf/tm1300_robot.urdf.xacro (robot description, xacro)
@@ -8,5 +8,5 @@
   <!-- tm1300 -->
   <xacro:include filename="$(find tm_description)/urdf/tm1300.urdf.xacro" />
-  <xacro:tm1300_robot prefix="${prefix}" joint_limited="false" />
+  <xacro:tm1300_robot prefix="${prefix}" joint_limited="false" has_camera="true" />
   <link name="world" />
   <joint name="world_joint" type="fixed">

File: tm_description/urdf/tm1300_robot_joint_limited.urdf.xacro (robot description, xacro)
@@ -8,5 +8,5 @@
   <!-- tm1300 -->
   <xacro:include filename="$(find tm_description)/urdf/tm1300.urdf.xacro" />
-  <xacro:tm1300_robot prefix="${prefix}" joint_limited="true" />
+  <xacro:tm1300_robot prefix="${prefix}" joint_limited="true" has_camera="true" />
   <link name="world" />
   <joint name="world_joint" type="fixed">

File: tm_description/urdf/tm700.urdf.xacro (robot description, xacro)
@@ -51,5 +51,5 @@
     </inertial>
   </xacro:macro>
-  <xacro:macro name="tm700_robot" params="prefix joint_limited">
+  <xacro:macro name="tm700_robot" params="prefix joint_limited has_camera">
     <!-- transmission prefix -->
     <xacro:tm_arm_transmission prefix="${prefix}" />
@@ -230,5 +230,10 @@
       <visual>
         <geometry>
-	  <mesh filename="package://tm_description/meshes/tm700/visual/Wrist3.STL" />
+          <xacro:if value="${has_camera}">
+          <mesh filename="package://tm_description/meshes/tm700/visual/Wrist3.STL" />
+          </xacro:if>
+          <xacro:unless value="${has_camera}">
+          <mesh filename="package://tm_description/meshes/tm700/visual/Wrist3_no_camera.STL" />
+          </xacro:unless>
         </geometry>
 	<origin xyz="0 0 0.015" rpy="0 0 0"/>
@@ -239,5 +244,10 @@
       <collision>
         <geometry>
-	  <mesh filename="package://tm_description/meshes/tm700/collision/wrist_3.STL" />
+          <xacro:if value="${has_camera}">
+	      <mesh filename="package://tm_description/meshes/tm700/collision/wrist_3.STL" />
+          </xacro:if>
+          <xacro:unless value="${has_camera}">
+	      <mesh filename="package://tm_description/meshes/tm700/collision/wrist_3_no_camera.STL" />
+          </xacro:unless>
         </geometry>
       </collision>

File: tm_description/urdf/tm700_robot.urdf.xacro (robot description, xacro)
@@ -8,5 +8,5 @@
   <!-- tm700 -->
   <xacro:include filename="$(find tm_description)/urdf/tm700.urdf.xacro" />
-  <xacro:tm700_robot prefix="${prefix}" joint_limited="false" />
+  <xacro:tm700_robot prefix="${prefix}" joint_limited="false" has_camera="true" />
   <link name="world" />
   <joint name="world_joint" type="fixed">

File: tm_description/urdf/tm700_robot_eih.urdf.xacro (robot description, xacro)
@@ -8,5 +8,5 @@
   <!-- tm700 -->
   <xacro:include filename="$(find tm_description)/urdf/tm700.urdf.xacro" />
-  <xacro:tm700_robot prefix="${prefix}" joint_limited="false" />
+  <xacro:tm700_robot prefix="${prefix}" joint_limited="false" has_camera="true" />
   <link name="world" />
   <joint name="world_joint" type="fixed">

File: tm_description/urdf/tm700_robot_joint_limited.urdf.xacro (robot description, xacro)
@@ -8,5 +8,5 @@
   <!-- tm700 -->
   <xacro:include filename="$(find tm_description)/urdf/tm700.urdf.xacro" />
-  <xacro:tm700_robot prefix="${prefix}" joint_limited="true" />
+  <xacro:tm700_robot prefix="${prefix}" joint_limited="true" has_camera="true"/>
   <link name="world" />
   <joint name="world_joint" type="fixed">

File: tm_description/urdf/tm700_robot_joint_limited_eih.urdf.xacro (robot description, xacro)
@@ -8,5 +8,5 @@
   <!-- tm700 -->
   <xacro:include filename="$(find tm_description)/urdf/tm700.urdf.xacro" />
-  <xacro:tm700_robot prefix="${prefix}" joint_limited="true" />
+  <xacro:tm700_robot prefix="${prefix}" joint_limited="true" has_camera="true" />
   <link name="world" />
   <joint name="world_joint" type="fixed">

File: tm_description/urdf/tm900.urdf.xacro (robot description, xacro)
@@ -50,5 +50,5 @@
     </inertial>
   </xacro:macro>
-  <xacro:macro name="tm900_robot" params="prefix joint_limited">
+  <xacro:macro name="tm900_robot" params="prefix joint_limited has_camera">
     <!-- transmission prefix -->
     <xacro:tm_arm_transmission prefix="${prefix}" />
@@ -229,5 +229,10 @@
       <visual>
         <geometry>
-	  <mesh filename="package://tm_description/meshes/tm900/visual/Wrist3.STL" />
+          <xacro:if value="${has_camera}">
+          <mesh filename="package://tm_description/meshes/tm900/visual/Wrist3.STL" />
+          </xacro:if>
+          <xacro:unless value="${has_camera}">
+          <mesh filename="package://tm_description/meshes/tm900/visual/Wrist3_no_camera.STL" />
+          </xacro:unless>
         </geometry>
 	<origin xyz="0 0 0.015" rpy="0 0 0"/>
@@ -238,5 +243,10 @@
       <collision>
         <geometry>
-	  <mesh filename="package://tm_description/meshes/tm900/collision/wrist_3.STL" />
+          <xacro:if value="${has_camera}">
+	      <mesh filename="package://tm_description/meshes/tm900/collision/wrist_3.STL" />
+          </xacro:if>
+          <xacro:unless value="${has_camera}">
+	      <mesh filename="package://tm_description/meshes/tm900/collision/wrist_3_no_camera.STL" />
+          </xacro:unless>
         </geometry>
       </collision>

File: tm_description/urdf/tm900_robot.urdf.xacro (robot description, xacro)
@@ -8,5 +8,5 @@
   <!-- tm900 -->
   <xacro:include filename="$(find tm_description)/urdf/tm900.urdf.xacro" />
-  <xacro:tm900_robot prefix="${prefix}" joint_limited="false" />
+  <xacro:tm900_robot prefix="${prefix}" joint_limited="false" has_camera="true" />
   <link name="world" />
   <joint name="world_joint" type="fixed">

File: tm_description/urdf/tm900_robot_eih.urdf.xacro (robot description, xacro)
@@ -8,5 +8,5 @@
   <!-- tm900 -->
   <xacro:include filename="$(find tm_description)/urdf/tm900.urdf.xacro" />
-  <xacro:tm900_robot prefix="${prefix}" joint_limited="false" />
+  <xacro:tm900_robot prefix="${prefix}" joint_limited="false" has_camera="true" />
   <link name="world" />
   <joint name="world_joint" type="fixed">

File: tm_description/urdf/tm900_robot_joint_limited.urdf.xacro (robot description, xacro)
@@ -8,5 +8,5 @@
   <!-- tm900 -->
   <xacro:include filename="$(find tm_description)/urdf/tm900.urdf.xacro" />
-  <xacro:tm900_robot prefix="${prefix}" joint_limited="true" />
+  <xacro:tm900_robot prefix="${prefix}" joint_limited="true" has_camera="true" />
   <link name="world" />
   <joint name="world_joint" type="fixed">

File: tm_description/urdf/tm900_robot_joint_limited_eih.urdf.xacro (robot description, xacro)
@@ -8,5 +8,5 @@
   <!-- tm900 -->
   <xacro:include filename="$(find tm_description)/urdf/tm900.urdf.xacro" />
-  <xacro:tm900_robot prefix="${prefix}" joint_limited="true" />
+  <xacro:tm900_robot prefix="${prefix}" joint_limited="true" has_camera="true" />
   <link name="world" />
   <joint name="world_joint" type="fixed">

Commit message: bugfix tm1100 xacro

File: tm_description/urdf/tm1100.urdf.xacro (robot description, xacro)
@@ -51,5 +51,5 @@
     </inertial>
   </xacro:macro>
-  <xacro:macro name="tm1100_robot" params="prefix joint_limited">
+  <xacro:macro name="tm1100_robot" params="prefix joint_limited has_camera">
     <!-- transmission prefix -->
     <xacro:tm_arm_transmission prefix="${prefix}" />
