Commit message: corrected joint and velocity limits

File: tm_description/urdf/tm1100.urdf.xacro (robot description, xacro)
@@ -96,8 +96,8 @@
       <axis xyz="0 -1 0" />
       <xacro:unless value="${joint_limited}">
-        <limit lower="${-2.0 * pi}" upper="${2.0 * pi}" effort="150.0" velocity="3.15"/>
-      </xacro:unless>
-      <xacro:if value="${joint_limited}">
-        <limit lower="${-pi}" upper="${pi}" effort="150.0" velocity="3.15"/>
+        <limit lower="${-270. / 180. * pi}" upper="${270. / 180. * pi}" effort="150.0" velocity="${120. / 180. * pi}"/>
+      </xacro:unless>
+      <xacro:if value="${joint_limited}">
+        <limit lower="${-pi}" upper="${pi}" effort="150.0" velocity="${120. / 180. * pi}"/>
       </xacro:if>
       <dynamics damping="0.0" friction="0.0"/>
@@ -127,8 +127,8 @@
       <axis xyz="0 0 1" />
       <xacro:unless value="${joint_limited}">
-        <limit lower="${-1.5 * pi}" upper="${1.5 * pi}" effort="150.0" velocity="3.15"/>
-      </xacro:unless>
-      <xacro:if value="${joint_limited}">
-        <limit lower="${-pi}" upper="${pi}" effort="150.0" velocity="3.15"/>
+        <limit lower="${-180. / 180. * pi}" upper="${180. / 180. * pi}" effort="150.0" velocity="${120. / 180. * pi}"/>
+      </xacro:unless>
+      <xacro:if value="${joint_limited}">
+        <limit lower="${-pi}" upper="${pi}" effort="150.0" velocity="${120. / 180. * pi}"/>
       </xacro:if>
       <dynamics damping="0.0" friction="0.0"/>
@@ -158,8 +158,8 @@
       <axis xyz="0 0 1" />
       <xacro:unless value="${joint_limited}">
-        <limit lower="${-1.5 * pi}" upper="${1.5 * pi}" effort="150.0" velocity="3.15"/>
-      </xacro:unless>
-      <xacro:if value="${joint_limited}">
-        <limit lower="${-pi}" upper="${pi}" effort="150.0" velocity="3.15"/>
+        <limit lower="${-163. / 180. * pi}" upper="${163. / 180. * pi}" effort="150.0" velocity="${150. / 180. * pi}"/>
+      </xacro:unless>
+      <xacro:if value="${joint_limited}">
+        <limit lower="${-pi}" upper="${pi}" effort="150.0" velocity="${180. / 180. * pi}"/>
       </xacro:if>
       <dynamics damping="0.0" friction="0.0"/>
@@ -189,8 +189,8 @@
       <axis xyz="0 1 0" />
       <xacro:unless value="${joint_limited}">
-        <limit lower="${-2.0 * pi}" upper="${2.0 * pi}" effort="28.0" velocity="3.2"/>
-      </xacro:unless>
-      <xacro:if value="${joint_limited}">
-        <limit lower="${-pi}" upper="${pi}" effort="28.0" velocity="3.2"/>
+        <limit lower="${-180. / 180. * pi}" upper="${180. / 180. * pi}" effort="28.0" velocity="${180. / 180. * pi}"/>
+      </xacro:unless>
+      <xacro:if value="${joint_limited}">
+        <limit lower="${-pi}" upper="${pi}" effort="28.0" velocity="${180. / 180. * pi}"/>
       </xacro:if>
       <dynamics damping="0.0" friction="0.0"/>
@@ -220,8 +220,8 @@
       <axis xyz="0 1 0" />
       <xacro:unless value="${joint_limited}">
-        <limit lower="${-2.0 * pi}" upper="${2.0 * pi}" effort="28.0" velocity="3.2"/>
-      </xacro:unless>
-      <xacro:if value="${joint_limited}">
-        <limit lower="${-pi}" upper="${pi}" effort="28.0" velocity="3.2"/>
+        <limit lower="${-180. / 180. * pi}" upper="${180. / 180. * pi}" effort="28.0" velocity="${180. / 180. * pi}"/>
+      </xacro:unless>
+      <xacro:if value="${joint_limited}">
+        <limit lower="${-pi}" upper="${pi}" effort="28.0" velocity="${180. / 180. * pi}"/>
       </xacro:if>
       <dynamics damping="0.0" friction="0.0"/>
@@ -262,8 +262,8 @@
       <axis xyz="0 0 1" />
       <xacro:unless value="${joint_limited}">
-        <limit lower="${-2.0 * pi}" upper="${2.0 * pi}" effort="28.0" velocity="3.2"/>
-      </xacro:unless>
-      <xacro:if value="${joint_limited}">
-        <limit lower="${-pi}" upper="${pi}" effort="28.0" velocity="3.2"/>
+        <limit lower="${-270. / 180. * pi}" upper="${270. / 180. * pi}" effort="28.0" velocity="${180. / 180. * pi}"/>
+      </xacro:unless>
+      <xacro:if value="${joint_limited}">
+        <limit lower="${-pi}" upper="${pi}" effort="28.0" velocity="${180. / 180. * pi}"/>
       </xacro:if>
       <dynamics damping="0.0" friction="0.0"/>

File: tm_description/urdf/tm1300.urdf.xacro (robot description, xacro)
@@ -95,8 +95,8 @@
       <axis xyz="0 -1 0" />
       <xacro:unless value="${joint_limited}">
-        <limit lower="${-2.0 * pi}" upper="${2.0 * pi}" effort="150.0" velocity="3.15"/>
-      </xacro:unless>
-      <xacro:if value="${joint_limited}">
-        <limit lower="${-pi}" upper="${pi}" effort="150.0" velocity="3.15"/>
+        <limit lower="${-270. / 180. * pi}" upper="${270. / 180. * pi}" effort="150.0" velocity="${120. / 180. * pi}"/>
+      </xacro:unless>
+      <xacro:if value="${joint_limited}">
+        <limit lower="${-pi}" upper="${pi}" effort="150.0" velocity="${120. / 180. * pi}"/>
       </xacro:if>
       <dynamics damping="0.0" friction="0.0"/>
@@ -126,8 +126,8 @@
       <axis xyz="0 0 1" />
       <xacro:unless value="${joint_limited}">
-        <limit lower="${-1.5 * pi}" upper="${1.5 * pi}" effort="150.0" velocity="3.15"/>
-      </xacro:unless>
-      <xacro:if value="${joint_limited}">
-        <limit lower="${-pi}" upper="${pi}" effort="150.0" velocity="3.15"/>
+        <limit lower="${-180. / 180. * pi}" upper="${180. / 180. * pi}" effort="150.0" velocity="${120. / 180. * pi}"/>
+      </xacro:unless>
+      <xacro:if value="${joint_limited}">
+        <limit lower="${-pi}" upper="${pi}" effort="150.0" velocity="${120. / 180. * pi}"/>
       </xacro:if>
       <dynamics damping="0.0" friction="0.0"/>
@@ -157,8 +157,8 @@
       <axis xyz="0 0 1" />
       <xacro:unless value="${joint_limited}">
-        <limit lower="${-1.5 * pi}" upper="${1.5 * pi}" effort="150.0" velocity="3.15"/>
-      </xacro:unless>
-      <xacro:if value="${joint_limited}">
-        <limit lower="${-pi}" upper="${pi}" effort="150.0" velocity="3.15"/>
+        <limit lower="${-166. / 180. * pi}" upper="${166. / 180. * pi}" effort="150.0" velocity="${180. / 180. * pi}"/>
+      </xacro:unless>
+      <xacro:if value="${joint_limited}">
+        <limit lower="${-pi}" upper="${pi}" effort="150.0" velocity="${180. / 180. * pi}"/>
       </xacro:if>
       <dynamics damping="0.0" friction="0.0"/>
@@ -188,8 +188,8 @@
       <axis xyz="0 1 0" />
       <xacro:unless value="${joint_limited}">
-        <limit lower="${-2.0 * pi}" upper="${2.0 * pi}" effort="28.0" velocity="3.2"/>
-      </xacro:unless>
-      <xacro:if value="${joint_limited}">
-        <limit lower="${-pi}" upper="${pi}" effort="28.0" velocity="3.2"/>
+        <limit lower="${-180. / 180. * pi}" upper="${180. / 180. * pi}" effort="28.0" velocity="${180. / 180. * pi}"/>
+      </xacro:unless>
+      <xacro:if value="${joint_limited}">
+        <limit lower="${-pi}" upper="${pi}" effort="28.0" velocity="${180. / 180. * pi}"/>
       </xacro:if>
       <dynamics damping="0.0" friction="0.0"/>
@@ -219,8 +219,8 @@
       <axis xyz="0 1 0" />
       <xacro:unless value="${joint_limited}">
-        <limit lower="${-2.0 * pi}" upper="${2.0 * pi}" effort="28.0" velocity="3.2"/>
-      </xacro:unless>
-      <xacro:if value="${joint_limited}">
-        <limit lower="${-pi}" upper="${pi}" effort="28.0" velocity="3.2"/>
+        <limit lower="${-180. / 180. * pi}" upper="${180. / 180. * pi}" effort="28.0" velocity="${180. / 180. * pi}"/>
+      </xacro:unless>
+      <xacro:if value="${joint_limited}">
+        <limit lower="${-pi}" upper="${pi}" effort="28.0" velocity="${180. / 180. * pi}"/>
       </xacro:if>
       <dynamics damping="0.0" friction="0.0"/>
@@ -261,8 +261,8 @@
       <axis xyz="0 0 1" />
       <xacro:unless value="${joint_limited}">
-        <limit lower="${-2.0 * pi}" upper="${2.0 * pi}" effort="28.0" velocity="3.2"/>
-      </xacro:unless>
-      <xacro:if value="${joint_limited}">
-        <limit lower="${-pi}" upper="${pi}" effort="28.0" velocity="3.2"/>
+        <limit lower="${-270. / 180. * pi}" upper="${270. / 180. * pi}" effort="28.0" velocity="${180. / 180. * pi}"/>
+      </xacro:unless>
+      <xacro:if value="${joint_limited}">
+        <limit lower="${-pi}" upper="${pi}" effort="28.0" velocity="${180. / 180. * pi}"/>
       </xacro:if>
       <dynamics damping="0.0" friction="0.0"/>

File: tm_description/urdf/tm700.urdf.xacro (robot description, xacro)
@@ -96,8 +96,8 @@
       <axis xyz="0 -1 0" />
       <xacro:unless value="${joint_limited}">
-        <limit lower="${-2.0 * pi}" upper="${2.0 * pi}" effort="150.0" velocity="3.15"/>
-      </xacro:unless>
-      <xacro:if value="${joint_limited}">
-        <limit lower="${-pi}" upper="${pi}" effort="150.0" velocity="3.15"/>
+        <limit lower="${-270. / 180. * pi}" upper="${270. / 180. * pi}" effort="150.0" velocity="${180 / 180. * pi}"/>
+      </xacro:unless>
+      <xacro:if value="${joint_limited}">
+        <limit lower="${-pi}" upper="${pi}" effort="150.0" velocity="${180 / 180. * pi}"/>
       </xacro:if>
       <dynamics damping="0.0" friction="0.0"/>
@@ -127,8 +127,8 @@
       <axis xyz="0 0 1" />
       <xacro:unless value="${joint_limited}">
-        <limit lower="${-1.5 * pi}" upper="${1.5 * pi}" effort="150.0" velocity="3.15"/>
-      </xacro:unless>
-      <xacro:if value="${joint_limited}">
-        <limit lower="${-pi}" upper="${pi}" effort="150.0" velocity="3.15"/>
+        <limit lower="${-180. / 180. * pi}" upper="${180. / 180. * pi}" effort="150.0" velocity="${180 / 180. * pi}"/>
+      </xacro:unless>
+      <xacro:if value="${joint_limited}">
+        <limit lower="${-pi}" upper="${pi}" effort="150.0" velocity="${180 / 180. * pi}"/>
       </xacro:if>
       <dynamics damping="0.0" friction="0.0"/>
@@ -157,10 +157,5 @@
       <origin xyz="${arm_1_length} 0.0 ${elbow_offset}" rpy="0.0 0.0 0.0" />
       <axis xyz="0 0 1" />
-      <xacro:unless value="${joint_limited}">
-        <limit lower="${-1.5 * pi}" upper="${1.5 * pi}" effort="150.0" velocity="3.15"/>
-      </xacro:unless>
-      <xacro:if value="${joint_limited}">
-        <limit lower="${-pi}" upper="${pi}" effort="150.0" velocity="3.15"/>
-      </xacro:if>
+      <limit lower="${-155. / 180. * pi}" upper="${155. / 180. * pi}" effort="150.0" velocity="${180 / 180. * pi}"/>
       <dynamics damping="0.0" friction="0.0"/>
     </joint>
@@ -189,8 +184,8 @@
       <axis xyz="0 1 0" />
       <xacro:unless value="${joint_limited}">
-        <limit lower="${-2.0 * pi}" upper="${2.0 * pi}" effort="28.0" velocity="3.2"/>
-      </xacro:unless>
-      <xacro:if value="${joint_limited}">
-        <limit lower="${-pi}" upper="${pi}" effort="28.0" velocity="3.2"/>
+        <limit lower="${-180. / 180. * pi}" upper="${180. / 180. * pi}" effort="28.0" velocity="${225. / 180. * pi}"/>
+      </xacro:unless>
+      <xacro:if value="${joint_limited}">
+        <limit lower="${-pi}" upper="${pi}" effort="28.0" velocity="${225. / 180. * pi}"/>
       </xacro:if>
       <dynamics damping="0.0" friction="0.0"/>
@@ -220,8 +215,8 @@
       <axis xyz="0 1 0" />
       <xacro:unless value="${joint_limited}">
-        <limit lower="${-2.0 * pi}" upper="${2.0 * pi}" effort="28.0" velocity="3.2"/>
-      </xacro:unless>
-      <xacro:if value="${joint_limited}">
-        <limit lower="${-pi}" upper="${pi}" effort="28.0" velocity="3.2"/>
+        <limit lower="${-180. / 180. * pi}" upper="${180. / 180. * pi}" effort="28.0" velocity="${225. / 180. * pi}"/>
+      </xacro:unless>
+      <xacro:if value="${joint_limited}">
+        <limit lower="${-pi}" upper="${pi}" effort="28.0" velocity="${225. / 180. * pi}"/>
       </xacro:if>
       <dynamics damping="0.0" friction="0.0"/>
@@ -262,8 +257,8 @@
       <axis xyz="0 0 1" />
       <xacro:unless value="${joint_limited}">
-        <limit lower="${-2.0 * pi}" upper="${2.0 * pi}" effort="28.0" velocity="3.2"/>
-      </xacro:unless>
-      <xacro:if value="${joint_limited}">
-        <limit lower="${-pi}" upper="${pi}" effort="28.0" velocity="3.2"/>
+        <limit lower="${-270. / 180. * pi}" upper="${270. / 180. * pi}" effort="28.0" velocity="${225. / 180. * pi}"/>
+      </xacro:unless>
+      <xacro:if value="${joint_limited}">
+        <limit lower="${-pi}" upper="${pi}" effort="28.0" velocity="${225. / 180. * pi}"/>
       </xacro:if>
       <dynamics damping="0.0" friction="0.0"/>

File: tm_description/urdf/tm900.urdf.xacro (robot description, xacro)
@@ -95,8 +95,8 @@
       <axis xyz="0 -1 0" />
       <xacro:unless value="${joint_limited}">
-        <limit lower="${-2.0 * pi}" upper="${2.0 * pi}" effort="150.0" velocity="3.15"/>
-      </xacro:unless>
-      <xacro:if value="${joint_limited}">
-        <limit lower="${-pi}" upper="${pi}" effort="150.0" velocity="3.15"/>
+        <limit lower="${-270. / 180. * pi}" upper="${270. / 180. * pi}" effort="150.0" velocity="${180 / 180. * pi}"/>
+      </xacro:unless>
+      <xacro:if value="${joint_limited}">
+        <limit lower="${-pi}" upper="${pi}" effort="150.0" velocity="${180 / 180. * pi}"/>
       </xacro:if>
       <dynamics damping="0.0" friction="0.0"/>
@@ -126,8 +126,8 @@
       <axis xyz="0 0 1" />
       <xacro:unless value="${joint_limited}">
-        <limit lower="${-1.5 * pi}" upper="${1.5 * pi}" effort="150.0" velocity="3.15"/>
-      </xacro:unless>
-      <xacro:if value="${joint_limited}">
-        <limit lower="${-pi}" upper="${pi}" effort="150.0" velocity="3.15"/>
+        <limit lower="${-180. / 180. * pi}" upper="${180. / 180. * pi}" effort="150.0" velocity="${180 / 180. * pi}"/>
+      </xacro:unless>
+      <xacro:if value="${joint_limited}">
+        <limit lower="${-pi}" upper="${pi}" effort="150.0" velocity="${180 / 180. * pi}"/>
       </xacro:if>
       <dynamics damping="0.0" friction="0.0"/>
@@ -156,10 +156,5 @@
       <origin xyz="${arm_1_length} 0.0 ${elbow_offset}" rpy="0.0 0.0 0.0" />
       <axis xyz="0 0 1" />
-      <xacro:unless value="${joint_limited}">
-        <limit lower="${-1.5 * pi}" upper="${1.5 * pi}" effort="150.0" velocity="3.15"/>
-      </xacro:unless>
-      <xacro:if value="${joint_limited}">
-        <limit lower="${-pi}" upper="${pi}" effort="150.0" velocity="3.15"/>
-      </xacro:if>
+      <limit lower="${-155. / 180. * pi}" upper="${155. / 180. * pi}" effort="150.0" velocity="${180 / 180. * pi}"/>
       <dynamics damping="0.0" friction="0.0"/>
     </joint>
@@ -188,8 +183,8 @@
       <axis xyz="0 1 0" />
       <xacro:unless value="${joint_limited}">
-        <limit lower="${-2.0 * pi}" upper="${2.0 * pi}" effort="28.0" velocity="3.2"/>
-      </xacro:unless>
-      <xacro:if value="${joint_limited}">
-        <limit lower="${-pi}" upper="${pi}" effort="28.0" velocity="3.2"/>
+        <limit lower="${-180. / 180. * pi}" upper="${180. / 180. * pi}" effort="28.0" velocity="${225. / 180. * pi}"/>
+      </xacro:unless>
+      <xacro:if value="${joint_limited}">
+        <limit lower="${-pi}" upper="${pi}" effort="28.0" velocity="${225. / 180. * pi}"/>
       </xacro:if>
       <dynamics damping="0.0" friction="0.0"/>
@@ -219,8 +214,8 @@
       <axis xyz="0 1 0" />
       <xacro:unless value="${joint_limited}">
-        <limit lower="${-2.0 * pi}" upper="${2.0 * pi}" effort="28.0" velocity="3.2"/>
-      </xacro:unless>
-      <xacro:if value="${joint_limited}">
-        <limit lower="${-pi}" upper="${pi}" effort="28.0" velocity="3.2"/>
+        <limit lower="${-180. / 180. * pi}" upper="${180. / 180. * pi}" effort="28.0" velocity="${225. / 180. * pi}"/>
+      </xacro:unless>
+      <xacro:if value="${joint_limited}">
+        <limit lower="${-pi}" upper="${pi}" effort="28.0" velocity="${225. / 180. * pi}"/>
       </xacro:if>
       <dynamics damping="0.0" friction="0.0"/>
@@ -261,8 +256,8 @@
       <axis xyz="0 0 1" />
       <xacro:unless value="${joint_limited}">
-        <limit lower="${-2.0 * pi}" upper="${2.0 * pi}" effort="28.0" velocity="3.2"/>
-      </xacro:unless>
-      <xacro:if value="${joint_limited}">
-        <limit lower="${-pi}" upper="${pi}" effort="28.0" velocity="3.2"/>
+        <limit lower="${-270. / 180. * pi}" upper="${270. / 180. * pi}" effort="28.0" velocity="${225. / 180. * pi}"/>
+      </xacro:unless>
+      <xacro:if value="${joint_limited}">
+        <limit lower="${-pi}" upper="${pi}" effort="28.0" velocity="${225. / 180. * pi}"/>
       </xacro:if>
       <dynamics damping="0.0" friction="0.0"/>
