Commit message: eliminated deprecated tag usage and pi being overwritten

File: tm_description/urdf/tm1100.urdf.xacro (robot description, xacro)
@@ -4,12 +4,11 @@
   <xacro:include filename="$(find tm_description)/urdf/tm.transmission.xacro" />
   <!-- Mass parameters -->
-  <property name="pi" value="3.14159265" />
-  <property name="base_mass" value="1.0" />
-  <property name="shoulder_mass" value="4.5" />
-  <property name="arm_1_mass" value="10.5" />
-  <property name="arm_2_mass" value="2.1" />
-  <property name="wrist_1_mass" value="1.45" />
-  <property name="wrist_2_mass" value="1.45" />
-  <property name="wrist_3_mass" value="0.4" />
+  <xacro:property name="base_mass" value="1.0" />
+  <xacro:property name="shoulder_mass" value="4.5" />
+  <xacro:property name="arm_1_mass" value="10.5" />
+  <xacro:property name="arm_2_mass" value="2.1" />
+  <xacro:property name="wrist_1_mass" value="1.45" />
+  <xacro:property name="wrist_2_mass" value="1.45" />
+  <xacro:property name="wrist_3_mass" value="0.4" />
   <!-- Kinematic model -->
   <!-- Properties from tmcontrol.conf -->
@@ -24,26 +23,26 @@
     center_of_mass = [ [0, -0.02561, 0.00193], [0.2125, 0, 0.11336], [0.11993, 0.0, 0.0265], [0, -0.0018, 0.01634], [0, 0.0018,0.01634], [0, 0, -0.001159] ]
   -->
-  <property name="tm_d1" value="0.1652" />
-  <property name="tm_a2" value="0.5361" />
-  <property name="tm_a3" value="0.4579" />
-  <property name="tm_d4" value="0.1563" />
-  <property name="tm_d5" value="0.1060" />
-  <property name="tm_d6" value="0.11315" />
+  <xacro:property name="tm_d1" value="0.1652" />
+  <xacro:property name="tm_a2" value="0.5361" />
+  <xacro:property name="tm_a3" value="0.4579" />
+  <xacro:property name="tm_d4" value="0.1563" />
+  <xacro:property name="tm_d5" value="0.1060" />
+  <xacro:property name="tm_d6" value="0.11315" />
   <!-- offsets for shoulder/elbow joints -->
-  <property name="shoulder_offset" value="-0.1801" />  <!-- measured from model -->
-  <property name="elbow_offset" value="0.1298" /> <!-- measured from model -->
-  <property name="wrist_offset" value="${-tm_d4 - elbow_offset - shoulder_offset}" />
+  <xacro:property name="shoulder_offset" value="-0.1801" />  <!-- measured from model -->
+  <xacro:property name="elbow_offset" value="0.1298" /> <!-- measured from model -->
+  <xacro:property name="wrist_offset" value="${-tm_d4 - elbow_offset - shoulder_offset}" />
   <!-- link lengths used in model -->
-  <property name="shoulder_height" value="${tm_d1}" />
-  <property name="arm_1_length" value="${tm_a2}" />
-  <property name="arm_2_length" value="${tm_a3}" />
-  <property name="wrist_1_length" value="tm_d5}" />
-  <property name="wrist_2_length" value="${tm_d5}" />
-  <property name="wrist_3_length" value="0.05525" />
-  <property name="ee_length" value="${tm_d6 - wrist_3_length}" />
+  <xacro:property name="shoulder_height" value="${tm_d1}" />
+  <xacro:property name="arm_1_length" value="${tm_a2}" />
+  <xacro:property name="arm_2_length" value="${tm_a3}" />
+  <xacro:property name="wrist_1_length" value="tm_d5}" />
+  <xacro:property name="wrist_2_length" value="${tm_d5}" />
+  <xacro:property name="wrist_3_length" value="0.05525" />
+  <xacro:property name="ee_length" value="${tm_d6 - wrist_3_length}" />
   <xacro:macro name="cylinder_inertial" params="radius length mass *origin">
     <inertial>
       <mass value="${mass}" />
-      <insert_block name="origin" />
+      <xacro:insert_block name="origin" />
       <inertia ixx="${0.0833333 * mass * (3 * radius * radius + length * length)}" ixy="0.0" ixz="0.0"
         iyy="${0.0833333 * mass * (3 * radius * radius + length * length)}" iyz="0.0"

File: tm_description/urdf/tm1300.urdf.xacro (robot description, xacro)
@@ -2,13 +2,12 @@
 <robot xmlns:xacro="http://www.ros.org/wiki/xacro">
   <xacro:include filename="$(find tm_description)/urdf/tm.transmission.xacro" />
-  <property name="pi" value="3.14159265" />
   <!-- Mass parameters-->
-  <property name="base_mass" value="1.0" />
-  <property name="shoulder_mass" value="4.5" />
-  <property name="arm_1_mass" value="11.0" />
-  <property name="arm_2_mass" value="2.5" />
-  <property name="wrist_1_mass" value="1.45" />
-  <property name="wrist_2_mass" value="1.45" />
-  <property name="wrist_3_mass" value="0.4" />
+  <xacro:property name="base_mass" value="1.0" />
+  <xacro:property name="shoulder_mass" value="4.5" />
+  <xacro:property name="arm_1_mass" value="11.0" />
+  <xacro:property name="arm_2_mass" value="2.5" />
+  <xacro:property name="wrist_1_mass" value="1.45" />
+  <xacro:property name="wrist_2_mass" value="1.45" />
+  <xacro:property name="wrist_3_mass" value="0.4" />
   <!-- Kinematic model -->
   <!-- Properties from tmcontrol.conf -->
@@ -23,26 +22,26 @@
     center_of_mass = [ [0, -0.02561, 0.00193], [0.2125, 0, 0.11336], [0.11993, 0.0, 0.0265], [0, -0.0018, 0.01634], [0, 0.0018,0.01634], [0, 0, -0.001159] ]
   -->
-  <property name="tm_d1" value="0.1652" />
-  <property name="tm_a2" value="0.6361" />
-  <property name="tm_a3" value="0.5579" />
-  <property name="tm_d4" value="0.1563" />
-  <property name="tm_d5" value="0.1060" />
-  <property name="tm_d6" value="0.11315" />
+  <xacro:property name="tm_d1" value="0.1652" />
+  <xacro:property name="tm_a2" value="0.6361" />
+  <xacro:property name="tm_a3" value="0.5579" />
+  <xacro:property name="tm_d4" value="0.1563" />
+  <xacro:property name="tm_d5" value="0.1060" />
+  <xacro:property name="tm_d6" value="0.11315" />
   <!-- offsets for shoulder/elbow joints -->
-  <property name="shoulder_offset" value="-0.1801" />  <!-- measured from model -->
-  <property name="elbow_offset" value="0.1298" /> <!-- measured from model -->
-  <property name="wrist_offset" value="${-tm_d4 - elbow_offset - shoulder_offset}" />
+  <xacro:property name="shoulder_offset" value="-0.1801" />  <!-- measured from model -->
+  <xacro:property name="elbow_offset" value="0.1298" /> <!-- measured from model -->
+  <xacro:property name="wrist_offset" value="${-tm_d4 - elbow_offset - shoulder_offset}" />
   <!-- link lengths used in model -->
-  <property name="shoulder_height" value="${tm_d1}" />
-  <property name="arm_1_length" value="${tm_a2}" />
-  <property name="arm_2_length" value="${tm_a3}" />
-  <property name="wrist_1_length" value="tm_d5}" />
-  <property name="wrist_2_length" value="${tm_d5}" />
-  <property name="wrist_3_length" value="0.05525" />
-  <property name="ee_length" value="${tm_d6 - wrist_3_length}" />
+  <xacro:property name="shoulder_height" value="${tm_d1}" />
+  <xacro:property name="arm_1_length" value="${tm_a2}" />
+  <xacro:property name="arm_2_length" value="${tm_a3}" />
+  <xacro:property name="wrist_1_length" value="tm_d5}" />
+  <xacro:property name="wrist_2_length" value="${tm_d5}" />
+  <xacro:property name="wrist_3_length" value="0.05525" />
+  <xacro:property name="ee_length" value="${tm_d6 - wrist_3_length}" />
   <xacro:macro name="cylinder_inertial" params="radius length mass *origin">
     <inertial>
       <mass value="${mass}" />
-      <insert_block name="origin" />
+      <xacro:insert_block name="origin" />
       <inertia ixx="${0.0833333 * mass * (3 * radius * radius + length * length)}" ixy="0.0" ixz="0.0"
         iyy="${0.0833333 * mass * (3 * radius * radius + length * length)}" iyz="0.0"

File: tm_description/urdf/tm700.urdf.xacro (robot description, xacro)
@@ -4,12 +4,11 @@
   <xacro:include filename="$(find tm_description)/urdf/tm.transmission.xacro" />
   <!-- Mass parameters -->
-  <property name="pi" value="3.14159265" />
-  <property name="base_mass" value="1.0" />
-  <property name="shoulder_mass" value="4.5" />
-  <property name="arm_1_mass" value="10.5" />
-  <property name="arm_2_mass" value="2.1" />
-  <property name="wrist_1_mass" value="1.45" />
-  <property name="wrist_2_mass" value="1.45" />
-  <property name="wrist_3_mass" value="0.4" />
+  <xacro:property name="base_mass" value="1.0" />
+  <xacro:property name="shoulder_mass" value="4.5" />
+  <xacro:property name="arm_1_mass" value="10.5" />
+  <xacro:property name="arm_2_mass" value="2.1" />
+  <xacro:property name="wrist_1_mass" value="1.45" />
+  <xacro:property name="wrist_2_mass" value="1.45" />
+  <xacro:property name="wrist_3_mass" value="0.4" />
   <!-- Kinematic model -->
   <!-- Properties from tmcontrol.conf -->
@@ -24,26 +23,26 @@
     center_of_mass = [ [0, -0.02561, 0.00193], [0.2125, 0, 0.11336], [0.11993, 0.0, 0.0265], [0, -0.0018, 0.01634], [0, 0.0018,0.01634], [0, 0, -0.001159] ](tm700)
   -->
-  <property name="tm_d1" value="0.1451" />
-  <property name="tm_a2" value="0.3290" />
-  <property name="tm_a3" value="0.3115" />
-  <property name="tm_d4" value="0.1222" />
-  <property name="tm_d5" value="0.1060" />
-  <property name="tm_d6" value="0.1144" />
+  <xacro:property name="tm_d1" value="0.1451" />
+  <xacro:property name="tm_a2" value="0.3290" />
+  <xacro:property name="tm_a3" value="0.3115" />
+  <xacro:property name="tm_d4" value="0.1222" />
+  <xacro:property name="tm_d5" value="0.1060" />
+  <xacro:property name="tm_d6" value="0.1144" />
   <!-- offsets for shoulder/elbow joints -->
-  <property name="shoulder_offset" value="-0.146" />  <!-- measured from model -->
-  <property name="elbow_offset" value="0.1298" /> <!-- measured from model -->
-  <property name="wrist_offset" value="${-tm_d4 - elbow_offset - shoulder_offset}" />
+  <xacro:property name="shoulder_offset" value="-0.146" />  <!-- measured from model -->
+  <xacro:property name="elbow_offset" value="0.1298" /> <!-- measured from model -->
+  <xacro:property name="wrist_offset" value="${-tm_d4 - elbow_offset - shoulder_offset}" />
   <!-- link lengths used in model -->
-  <property name="shoulder_height" value="${tm_d1}" />
-  <property name="arm_1_length" value="${tm_a2}" />
-  <property name="arm_2_length" value="${tm_a3}" />
-  <property name="wrist_1_length" value="tm_d5}" />
-  <property name="wrist_2_length" value="${tm_d5}" />
-  <property name="wrist_3_length" value="0.0565" />
-  <property name="ee_length" value="${tm_d6 - wrist_3_length}" />
+  <xacro:property name="shoulder_height" value="${tm_d1}" />
+  <xacro:property name="arm_1_length" value="${tm_a2}" />
+  <xacro:property name="arm_2_length" value="${tm_a3}" />
+  <xacro:property name="wrist_1_length" value="tm_d5}" />
+  <xacro:property name="wrist_2_length" value="${tm_d5}" />
+  <xacro:property name="wrist_3_length" value="0.0565" />
+  <xacro:property name="ee_length" value="${tm_d6 - wrist_3_length}" />
   <xacro:macro name="cylinder_inertial" params="radius length mass *origin">
     <inertial>
       <mass value="${mass}" />
-      <insert_block name="origin" />
+      <xacro:insert_block name="origin" />
       <inertia ixx="${0.0833333 * mass * (3 * radius * radius + length * length)}" ixy="0.0" ixz="0.0"
         iyy="${0.0833333 * mass * (3 * radius * radius + length * length)}" iyz="0.0"

File: tm_description/urdf/tm900.urdf.xacro (robot description, xacro)
@@ -2,13 +2,12 @@
 <robot xmlns:xacro="http://www.ros.org/wiki/xacro">
   <xacro:include filename="$(find tm_description)/urdf/tm.transmission.xacro" />
-  <property name="pi" value="3.14159265" />
   <!-- Mass parameters-->
-  <property name="base_mass" value="1.0" />
-  <property name="shoulder_mass" value="4.5" />
-  <property name="arm_1_mass" value="11.0" />
-  <property name="arm_2_mass" value="2.5" />
-  <property name="wrist_1_mass" value="1.45" />
-  <property name="wrist_2_mass" value="1.45" />
-  <property name="wrist_3_mass" value="0.4" />
+  <xacro:property name="base_mass" value="1.0" />
+  <xacro:property name="shoulder_mass" value="4.5" />
+  <xacro:property name="arm_1_mass" value="11.0" />
+  <xacro:property name="arm_2_mass" value="2.5" />
+  <xacro:property name="wrist_1_mass" value="1.45" />
+  <xacro:property name="wrist_2_mass" value="1.45" />
+  <xacro:property name="wrist_3_mass" value="0.4" />
   <!-- Kinematic model -->
   <!-- Properties from tmcontrol.conf -->
@@ -23,26 +22,26 @@
     center_of_mass = [ [0, -0.02561, 0.00193], [0.2125, 0, 0.11336], [0.11993, 0.0, 0.0265], [0, -0.0018, 0.01634], [0, 0.0018,0.01634], [0, 0, -0.001159] ](tm900)
   -->
-  <property name="tm_d1" value="0.1451" />
-  <property name="tm_a2" value="0.4290" />
-  <property name="tm_a3" value="0.4115" />
-  <property name="tm_d4" value="0.1222" />
-  <property name="tm_d5" value="0.1060" />
-  <property name="tm_d6" value="0.1144" />
+  <xacro:property name="tm_d1" value="0.1451" />
+  <xacro:property name="tm_a2" value="0.4290" />
+  <xacro:property name="tm_a3" value="0.4115" />
+  <xacro:property name="tm_d4" value="0.1222" />
+  <xacro:property name="tm_d5" value="0.1060" />
+  <xacro:property name="tm_d6" value="0.1144" />
   <!-- offsets for shoulder/elbow joints -->
-  <property name="shoulder_offset" value="-0.146" />  <!-- measured from model -->
-  <property name="elbow_offset" value="0.1298" /> <!-- measured from model -->
-  <property name="wrist_offset" value="${-tm_d4 - elbow_offset - shoulder_offset}" />
+  <xacro:property name="shoulder_offset" value="-0.146" />  <!-- measured from model -->
+  <xacro:property name="elbow_offset" value="0.1298" /> <!-- measured from model -->
+  <xacro:property name="wrist_offset" value="${-tm_d4 - elbow_offset - shoulder_offset}" />
   <!-- link lengths used in model -->
-  <property name="shoulder_height" value="${tm_d1}" />
-  <property name="arm_1_length" value="${tm_a2}" />
-  <property name="arm_2_length" value="${tm_a3}" />
-  <property name="wrist_1_length" value="tm_d5}" />
-  <property name="wrist_2_length" value="${tm_d5}" />
-  <property name="wrist_3_length" value="0.0565" />
-  <property name="ee_length" value="${tm_d6 - wrist_3_length}" />
+  <xacro:property name="shoulder_height" value="${tm_d1}" />
+  <xacro:property name="arm_1_length" value="${tm_a2}" />
+  <xacro:property name="arm_2_length" value="${tm_a3}" />
+  <xacro:property name="wrist_1_length" value="tm_d5}" />
+  <xacro:property name="wrist_2_length" value="${tm_d5}" />
+  <xacro:property name="wrist_3_length" value="0.0565" />
+  <xacro:property name="ee_length" value="${tm_d6 - wrist_3_length}" />
   <xacro:macro name="cylinder_inertial" params="radius length mass *origin">
     <inertial>
       <mass value="${mass}" />
-      <insert_block name="origin" />
+      <xacro:insert_block name="origin" />
       <inertia ixx="${0.0833333 * mass * (3 * radius * radius + length * length)}" ixy="0.0" ixz="0.0"
         iyy="${0.0833333 * mass * (3 * radius * radius + length * length)}" iyz="0.0"

Commit message: remove extra collision box in tip_link; remove extra unused urdf eih files

File: tm_description/urdf/tm1100.urdf.xacro (robot description, xacro)
@@ -268,12 +268,5 @@
       <dynamics damping="0.0" friction="0.0"/>
     </joint>
-    <link name="${prefix}tip_link">
-      <collision>
-        <geometry>
-          <box size="0.05 0.05 0.05"/>
-        </geometry>
-        <origin xyz="0 0 0.025" rpy="0 0 0"/>
-      </collision>
-    </link>
+    <link name="${prefix}tip_link"/>
     <joint name="${prefix}tip_fixed_joint" type="fixed">
       <parent link="${prefix}wrist_3_link" />

File: tm_description/urdf/tm1300.urdf.xacro (robot description, xacro)
@@ -267,12 +267,5 @@
       <dynamics damping="0.0" friction="0.0"/>
     </joint>
-    <link name="${prefix}tip_link">
-      <collision>
-        <geometry>
-          <box size="0.05 0.05 0.05"/>
-        </geometry>
-        <origin xyz="0 0 0.025" rpy="0 0 0"/>
-      </collision>
-    </link>
+    <link name="${prefix}tip_link"/>
     <joint name="${prefix}tip_fixed_joint" type="fixed">
       <parent link="${prefix}wrist_3_link" />

File: tm_description/urdf/tm700.urdf.xacro (robot description, xacro)
@@ -263,12 +263,5 @@
       <dynamics damping="0.0" friction="0.0"/>
     </joint>
-    <link name="${prefix}tip_link">
-      <collision>
-        <geometry>
-          <box size="0.05 0.05 0.05"/>
-        </geometry>
-        <origin xyz="0 0 0.025" rpy="0 0 0"/>
-      </collision>
-    </link>
+    <link name="${prefix}tip_link"/>
     <joint name="${prefix}tip_fixed_joint" type="fixed">
       <parent link="${prefix}wrist_3_link" />

File: tm_description/urdf/tm900.urdf.xacro (robot description, xacro)
@@ -262,12 +262,5 @@
       <dynamics damping="0.0" friction="0.0"/>
     </joint>
-    <link name="${prefix}tip_link">
-      <collision>
-        <geometry>
-          <box size="0.05 0.05 0.05"/>
-        </geometry>
-        <origin xyz="0 0 0.025" rpy="0 0 0"/>
-      </collision>
-    </link>
+    <link name="${prefix}tip_link"/>
     <joint name="${prefix}tip_fixed_joint" type="fixed">
       <parent link="${prefix}wrist_3_link" />
